File: pic16f84_test.sch (KiCad schematic (older format))
At the start: 20 parts, among them J1 ICSP, J2 Conn_01x03, Q1 2N7002, Q2 2N7002, Q3 2N7002, Q4 2N7002, U1 PIC16F54-IP

Commit message: done with revision 0.01
Parts:
- added H1, H2, H3, H4: MountingHole, MountingHole:MountingHole_2.2mm_M2, symbol Mechanical:MountingHole
- J1: symbol custom:ICSP -> pic16f84_test-rescue:ICSP-custom
Connections:
- net SEG_F is gone; now on net PGC: AFF1.9 (f), AFF2.9 (f), AFF3.9 (f), AFF4.9 (f), U1.12 (ICSPCLK/RB6)
- net SEG_G is gone; now on net PGD: AFF1.10 (g), AFF2.10 (g), AFF3.10 (g), AFF4.10 (g), U1.13 (ICSPDAT/RB7)
Changed lines of the file:
@@
 $EndDescr
 $Comp
-L custom:ICSP J1
+L pic16f84_test-rescue:ICSP-custom J1
 U 1 1 5EE8F0E9
 P 2700 1950
@@
 Wire Wire Line
 	5900 4750 6700 4750
+$Comp
+L Mechanical:MountingHole H1
+U 1 1 5EF8E59E
+P 2400 6050
+F 0 "H1" H 2500 6096 50  0000 L CNN
+F 1 "MountingHole" H 2500 6005 50  0000 L CNN
+F 2 "MountingHole:MountingHole_2.2mm_M2" H 2400 6050 50  0001 C CNN
+F 3 "~" H 2400 6050 50  0001 C CNN
+	1    2400 6050
+	1    0    0    -1
+$EndComp
+$Comp
+L Mechanical:MountingHole H2
+U 1 1 5EF8E867
+P 2400 6250
+F 0 "H2" H 2500 6296 50  0000 L CNN
+F 1 "MountingHole" H 2500 6205 50  0000 L CNN
+F 2 "MountingHole:MountingHole_2.2mm_M2" H 2400 6250 50  0001 C CNN
+F 3 "~" H 2400 6250 50  0001 C CNN
+	1    2400 6250
+	1    0    0    -1
+$EndComp
+$Comp
+L Mechanical:MountingHole H3
+U 1 1 5EF8E8A7
+P 2400 6450
+F 0 "H3" H 2500 6496 50  0000 L CNN
+F 1 "MountingHole" H 2500 6405 50  0000 L CNN
+F 2 "MountingHole:MountingHole_2.2mm_M2" H 2400 6450 50  0001 C CNN
+F 3 "~" H 2400 6450 50  0001 C CNN
+	1    2400 6450
+	1    0    0    -1
+$EndComp
+$Comp
+L Mechanical:MountingHole H4
+U 1 1 5EF8E8E9
+P 2400 6650
+F 0 "H4" H 2500 6696 50  0000 L CNN
+F 1 "MountingHole" H 2500 6605 50  0000 L CNN
+F 2 "MountingHole:MountingHole_2.2mm_M2" H 2400 6650 50  0001 C CNN
+F 3 "~" H 2400 6650 50  0001 C CNN
+	1    2400 6650
+	1    0    0    -1
+$EndComp
+Text Label 6250 4650 2    50   ~ 0
+PGC
+Text Label 6250 4750 2    50   ~ 0
+PGD
 $EndSCHEMATC

Commit message: augment the diameter of the mounting holes
Parts:
- H1, H2, H3, H4: footprint MountingHole:MountingHole_2.2mm_M2 -> modules:MountingHole_3.2mm_M2
Changed lines of the file:
@@
 F 0 "H1" H 2500 6096 50  0000 L CNN
 F 1 "MountingHole" H 2500 6005 50  0000 L CNN
-F 2 "MountingHole:MountingHole_2.2mm_M2" H 2400 6050 50  0001 C CNN
+F 2 "modules:MountingHole_3.2mm_M2" H 2400 6050 50  0001 C CNN
 F 3 "~" H 2400 6050 50  0001 C CNN
 	1    2400 6050
@@
 F 0 "H2" H 2500 6296 50  0000 L CNN
 F 1 "MountingHole" H 2500 6205 50  0000 L CNN
-F 2 "MountingHole:MountingHole_2.2mm_M2" H 2400 6250 50  0001 C CNN
+F 2 "modules:MountingHole_3.2mm_M2" H 2400 6250 50  0001 C CNN
 F 3 "~" H 2400 6250 50  0001 C CNN
 	1    2400 6250
@@
 F 0 "H3" H 2500 6496 50  0000 L CNN
 F 1 "MountingHole" H 2500 6405 50  0000 L CNN
-F 2 "MountingHole:MountingHole_2.2mm_M2" H 2400 6450 50  0001 C CNN
+F 2 "modules:MountingHole_3.2mm_M2" H 2400 6450 50  0001 C CNN
 F 3 "~" H 2400 6450 50  0001 C CNN
 	1    2400 6450
@@
 F 0 "H4" H 2500 6696 50  0000 L CNN
 F 1 "MountingHole" H 2500 6605 50  0000 L CNN
-F 2 "MountingHole:MountingHole_2.2mm_M2" H 2400 6650 50  0001 C CNN
+F 2 "modules:MountingHole_3.2mm_M2" H 2400 6650 50  0001 C CNN
 F 3 "~" H 2400 6650 50  0001 C CNN
 	1    2400 6650

Commit message: just 3 segments
Parts:
- removed AFF4: LTS-6980HR, Display_7Segment:7SegmentLED_LTS6760_LTS6780, symbol Display_Character:LTS-6980HR
- removed Q4: 2N7002, Package_TO_SOT_SMD:SOT-23, symbol Transistor_FET:2N7002
- added J3: Conn_01x03, Connector_PinHeader_2.54mm:PinHeader_1x03_P2.54mm_Vertical, symbol Connector_Generic:Conn_01x03
- added R10, R2, R8, R9: 100, Resistor_SMD:R_0603_1608Metric_Pad1.05x0.95mm_HandSolder, symbol Device:R_Small
Connections:
- net DIG_3 is gone; now on net DIO: U1.2 (RA3)
- net DIO: now also J3.2 (Pin_2); no longer U1.6 (RB0)
- net GND: now also J3.1 (Pin_1)
- net PGC: now also J1.5 (PGC), R9.2; no longer AFF1.9 (f), AFF2.9 (f), AFF3.9 (f), J1.4 (PGD)
- net PGD: now also J1.4 (PGD), R10.2; no longer AFF1.10 (g), AFF2.10 (g), AFF3.10 (g), J1.5 (PGC)
- net SEG_A: now also R4.1; no longer U1.7 (RB1)
- net SEG_B: now also R5.1; no longer U1.8 (RB2)
- net SEG_C: now also R6.1; no longer U1.9 (RB3)
- net SEG_D: now also R7.1; no longer U1.10 (RB4)
- net SEG_E: now also R2.1; no longer U1.11 (RB5)
- net VCC: now also J3.3 (Pin_3)
- net at R4.2: now also U1.6 (RB0); no longer AFF1.3 (C.K.)
- net SEG_DP: now reaches AFF1.5 (DP)
- net SEG_DP: now also AFF2.5 (DP), AFF3.5 (DP), R10.1
- net at R5.2: now also U1.7 (RB1); no longer AFF2.3 (C.K.)
- net at R6.2: now also U1.8 (RB2); no longer AFF3.3 (C.K.)
- net at R7.2: now also U1.9 (RB3)
- net at Q1.3 (D): now also AFF1.3 (C.K.); no longer R4.1
- net at Q2.3 (D): now also AFF2.3 (C.K.); no longer R5.1
- net at Q3.3 (D): now also AFF3.3 (C.K.); no longer R6.1
- new net: R2.2, U1.10 (RB4)
- new net: R8.2, U1.11 (RB5)
- new net SEG_F: AFF1.9 (f), AFF2.9 (f), AFF3.9 (f), R8.1
- new net SEG_G: AFF1.10 (g), AFF2.10 (g), AFF3.10 (g), R9.1
Other:
- moved on the sheet: AFF1, AFF2, AFF3, Q1, Q2, Q3, R4, R5, R6, R7
